File: Mainboard/Mainboard.kicad_pcb (KiCad board)
At the start: 4 copper layers, 78.8 x 40 mm, 123 parts, among them IC1 IP5306, IC6 XC7S50-L1CSGA324I, J1 2479774-2, J3 Conn_01x06_Pin, J4 Left Daughter Connector, J5 Right Daughter Connector, J6 CART, J9 Screen zif FFC/FPC, SW1 POW, U1 LM3880, U2 MAX98357A, U3 TPS22917DBV, U4 TLV62569DBV, U5 W25Q128JVS, U6 TLV75518PDBV, U7 TPS62822DLC

Commit message: right daughter card added
Parts:
- removed the DR at (148.9, 85.5)
Connections:
- IC6 pad H18: Net-(IC6-IO_L21P_T3_DQS_15) -> (no net)
- J5 pad 1: Net-(IC6-IO_L21P_T3_DQS_15) -> VREF3V3
Routing:
- net Net-(IC6-IO_L21P_T3_DQS_15): track 34.9 -> 0.00 mm
- net VREF3V3: track 132.4 -> 158.1 mm, vias 27 -> 28
