File: Mainboard/_restore_backup_2026-07-22T16-07-43-759/Mainboard.kicad_sch (KiCad schematic)
At the start: 0 parts

Commit message: + Power sw, + R arrays, sync PCB/schem
Other:
- added sheet Screen (screen.kicad_sch)
Changed lines of the file:
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@@
 	(paper "A4")
 	(sheet
-		(at 143.51 36.83)
+		(at 182.88 35.56)
 		(size 36.83 25.4)
 		(exclude_from_sim no)
@@
 		)
 		(property "Sheetname" "FPGA"
-			(at 143.51 36.1184 0)
+			(at 182.88 34.8484 0)
 			(show_name no)
 			(do_not_autoplace no)
@@
 		)
 		(property "Sheetfile" "fpga_sch.kicad_sch"
-			(at 143.51 62.8146 0)
+			(at 182.88 61.5446 0)
 			(show_name no)
 			(do_not_autoplace no)
@@
 				)
 			)
+		)
+	)
+	(sheet
+		(at 30.48 81.28)
+		(size 34.29 22.86)
+		(exclude_from_sim no)
+		(in_bom yes)
+		(on_board yes)
+		(dnp no)
+		(fields_autoplaced yes)
+		(stroke
+			(width 0.1524)
+			(type solid)
+		)
+		(fill
+			(color 0 0 0 0)
+		)
+		(property "Sheetname" "Screen"
+			(at 30.48 80.5684 0)
+			(show_name no)
+			(do_not_autoplace no)
+			(effects
+				(font
+					(size 1.27 1.27)
+				)
+				(justify left bottom)
+			)
+		)
+		(property "Sheetfile" "screen.kicad_sch"
+			(at 30.48 104.7246 0)
+			(show_name no)
+			(do_not_autoplace no)
+			(effects
+				(font
+					(size 1.27 1.27)
+				)
+				(justify left top)
+			)
+		)
+		(instances
+			(project "Mainboard"
+				(path "/53a66bf0-ca24-4129-bc39-ed3123c0a797"
+					(page "5")
+				)
+			)
